Commit message: Fix link orientations

File: src/uh_simulation/person_sim/urdf/person.xacro (robot description, xacro)
@@ -107,8 +107,8 @@
 		</xacro:arm>
 		<xacro:arm name="${name}_arm_left" parent="${name}_shoulders">
-			<origin rpy="0 0 0" xyz="-0.23 0 -0.05" />
+			<origin rpy="0 0 3.14159" xyz="-0.23 0 -0.05" />
 		</xacro:arm>
 		<xacro:head name="${name}_head" parent="${name}_shoulders">
-			<origin rpy="0 0 0" xyz="0 0 0.07" />
+			<origin rpy="0 0 -1.57079" xyz="0 0 0.07" />
 		</xacro:head>
 	</xacro:macro>
@@ -265,14 +265,14 @@
 	</xacro:leg>
 	<xacro:wheel name="front_right" parent="base" reflect="1">
+		<origin rpy="0 0 0" xyz=" 0.1 -0.18 0" />
+	</xacro:wheel>
+	<xacro:wheel name="rear_right" parent="base" reflect="1">
+		<origin rpy="0 0 0" xyz="-0.1 -0.18 0" />
+	</xacro:wheel>
+	<xacro:wheel name="front_left" parent="base" reflect="-1">
+		<origin rpy="0 0 0" xyz="0.1 0.18 0" />
+	</xacro:wheel>
+	<xacro:wheel name="rear_left" parent="base" reflect="-1">
 		<origin rpy="0 0 0" xyz=" -0.1 0.18 0" />
-	</xacro:wheel>
-	<xacro:wheel name="rear_right" parent="base" reflect="1">
-		<origin rpy="0 0 0" xyz="0.1 0.18 0" />
-	</xacro:wheel>
-	<xacro:wheel name="front_left" parent="base" reflect="-1">
-		<origin rpy="0 0 0" xyz="-0.1 -0.18 0" />
-	</xacro:wheel>
-	<xacro:wheel name="rear_left" parent="base" reflect="-1">
-		<origin rpy="0 0 0" xyz=" 0.1 -0.18 0" />
 	</xacro:wheel>
 	<gazebo>

Commit message: cleanup WB->Ros conversions. Return 3D RPY locations data on SF.  Add 'hair' as direction indicator for person.

File: src/uh_simulation/person_sim/urdf/person.xacro (robot description, xacro)
@@ -10,5 +10,5 @@
 	<xacro:macro name="wheel" params="name parent reflect *origin">
 		<link name="${parent}_${name}_wheel">
-			<inertial>
+			<!-- inertial>
 				<mass value="0.5" />
 				<origin xyz="0 0 0" rpy="${-3.1415927/2} 0 0" />
@@ -30,9 +30,9 @@
 					<cylinder radius="0.1" length="0.02" />
 				</geometry>
-			</collision>
-		</link>
-		<gazebo reference="${parent}_${name}_wheel">
+			</collision-->
+		</link>
+		<!-- gazebo reference="${parent}_${name}_wheel">
 			<material value="Gazebo/Black" />
-		</gazebo>
+		</gazebo-->
 		<joint name="${parent}_${name}_wheel_joint" type="continuous">
 			<axis xyz="0 1 0" />
@@ -181,4 +181,7 @@
 			</collision>
 		</link>
+		<xacro:hair name="${name}_hair" parent="${name}">
+			<origin xyz="-0.02 0 0.02" rpy="0 0 0" />
+		</xacro:hair>
 		<gazebo reference="${name}_bottom_link">
 			<material>Gazebo/Grey</material>
@@ -189,4 +192,82 @@
 		<gazebo reference="${name}_top_link">
 			<material>Gazebo/Grey</material>
+		</gazebo>
+	</xacro:macro>
+	<xacro:macro name="hair" params="name parent *origin">
+		<joint name="${name}_bottom_joint" type="fixed">
+			<insert_block name="origin" />
+			<parent link="${parent}_link" />
+			<child link="${name}_link" />
+		</joint>
+		<link name="${name}_link">
+		</link>
+		<joint name="${name}_joint" type="fixed">
+			<origin xyz="0 0 0.08" rpy="0 0 0" />
+			<parent link="${name}_link" />
+			<child link="${name}_bottom_link" />
+		</joint>
+		<link name="${name}_bottom_link">
+			<visual>
+				<geometry>
+					<sphere radius="0.08" />
+				</geometry>
+				<material name="hair">
+					<color rgba="0.28 0.28 0.28 1.0" />
+				</material>
+			</visual>
+			<collision>
+				<geometry>
+					<sphere radius="0.08" />
+				</geometry>
+			</collision>
+		</link>
+		<joint name="${name}_middle_joint" type="fixed">
+			<origin xyz="0 0 0.035" rpy="0 0 0" />
+			<parent link="${name}_bottom_link" />
+			<child link="${name}_middle_link" />
+		</joint>
+		<link name="${name}_middle_link">
+			<visual>
+				<geometry>
+					<cylinder length="0.07" radius="0.08" />
+				</geometry>
+				<material name="hair">
+					<color rgba="0.28 0.28 0.28 1.0" />
+				</material>
+			</visual>
+			<collision>
+				<geometry>
+					<cylinder length="0.07" radius="0.08" />
+				</geometry>
+			</collision>
+		</link>
+		<joint name="${name}_top_joint" type="fixed">
+			<origin xyz="0 0 0.15" rpy="0 0 0" />
+			<parent link="${name}_link" />
+			<child link="${name}_top_link" />
+		</joint>
+		<link name="${name}_top_link">
+			<visual>
+				<geometry>
+					<sphere radius="0.08" />
+				</geometry>
+				<material name="hair">
+					<color rgba="0.28 0.28 0.28 1.0" />
+				</material>
+			</visual>
+			<collision>
+				<geometry>
+					<sphere radius="0.08" />
+				</geometry>
+			</collision>
+		</link>
+		<gazebo reference="${name}_bottom_link">
+			<material>Gazebo/Grey</material>
+		</gazebo>
+		<gazebo reference="${name}_middle_link">
+			<material>Gazebo/Black</material>
+		</gazebo>
+		<gazebo reference="${name}_top_link">
+			<material>Gazebo/Black</material>
 		</gazebo>
 	</xacro:macro>
