Commit message: Add source files, cleanup duplicate textures, fix gazebo launch

File: src/uh_environments/uh-robot-house/urdf/world.urdf.xacro (robot description, xacro)
@@ -31,6 +31,7 @@
 		</inertial>
 		<collision name="floor_collision">
+			<origin xyz="-1.8 2.15 0" />
 			<geometry>
-				<mesh filename="package://uh_environments/uh-robot-house/models/robot_house_ground.dae" />
+				<box size="10.5 10.5 0" />
 			</geometry>
 		</collision>

Commit message: Updates to world model, work around gazebo dae collision problem

File: src/uh_environments/uh-robot-house/urdf/world.urdf.xacro (robot description, xacro)
@@ -1,6 +1,6 @@
-<?xml version="1.0" ?>
-<robot xmlns:sensor="http://playerstage.sourceforge.net/gazebo/xmlschema/#sensor" xmlns:controller="http://playerstage.sourceforge.net/gazebo/xmlschema/#controller"
-	xmlns:interface="http://playerstage.sourceforge.net/gazebo/xmlschema/#interface" xmlns:xacro="http://playerstage.sourceforge.net/gazebo/xmlschema/#interface"
-	name="robot_house">
+<?xml version="1.0"?>
+<robot name="robot_house" xmlns:xacro="http://www.ros.org/wiki/xacro">
+	<xacro:include filename="$(find uh_environments)/uh-robot-house/urdf/world_ground.urdf.xacro" />
+	<xacro:include filename="$(find uh_environments)/uh-robot-house/urdf/world_walls.urdf.xacro" />
 	<gazebo>
 		<static>true</static>
@@ -11,42 +11,9 @@
 	</gazebo>
 	<link name="world" />
-	<joint name="ground_fixed" type="fixed">
-		<parent link="world" />
-		<child link="robot_house_ground" />
-	</joint>
-	<joint name="walls_fixed" type="fixed">
-		<parent link="robot_house_ground" />
-		<child link="robot_house_walls" />
-	</joint>
-	<link name="robot_house_ground">
-		<visual name="floor_visual">
-			<cast_shadows>false</cast_shadows>
-			<geometry>
-				<mesh filename="package://uh_environments/uh-robot-house/models/robot_house_ground.dae" />
-			</geometry>
-		</visual>
-		<inertial>
-			<mass value="1000" />
-			<inertia ixx="0" ixy="0" ixz="0" iyy="0" iyz="0" izz="0" />
-		</inertial>
-		<collision name="floor_collision">
-			<origin xyz="-1.8 2.15 0" />
-			<geometry>
-				<box size="10.5 10.5 0" />
-			</geometry>
-		</collision>
-	</link>
-	<link name="robot_house_walls">
-		<visual name="walls_visual">
-			<cast_shadows>false</cast_shadows>
-			<geometry>
-				<mesh filename="package://uh_environments/uh-robot-house/models/robot_house_walls.dae" />
-			</geometry>
-		</visual>
-		<collision name="walls_collision">
-			<geometry>
-				<mesh filename="package://uh_environments/uh-robot-house/models/robot_house_walls.dae" />
-			</geometry>
-		</collision>
-	</link>
+	<xacro:ground name="ground" parent="world">
+		<origin rpy="0 0 0" xyz="0 0 0" />
+	</xacro:ground>
+	<xacro:walls name="walls" parent="world">
+		<origin rpy="0 0 0" xyz="0 0 0" />
+	</xacro:walls>
 </robot>
